File: Bodensensor-KiCAD/Bodensensor.sch (KiCad schematic (older format))
At the start: 3 parts, among them IC1 4046

Commit message: added 2x5 pin connector symbol
Parts:
- added P1: CONN_02X05, symbol CONN_02X05
- added R1, R? (x7): 100R, symbol R_Small
Connections:
- net +3V3: now also P1.10 (P10)
- net GND: now also P1.9 (P9)
- net OUT: now also R1.1, R?.1, R?.1, R?.1, R?.2, R?.2, R?.2, R?.2
- new net: P1.1 (P1), R?.1
- new net: P1.2 (P2), R1.2
- new net: P1.3 (P3), R?.1
- new net: P1.4 (P4), R?.2
- new net: P1.5 (P5), R?.1
- new net: P1.6 (P6), R?.2
- new net: P1.7 (P7), R?.1
- new net: P1.8 (P8), R?.2
Changed lines of the file:
@@
 	1    0    0    -1
 $EndComp
-Wire Wire Line
-	4950 4100 4650 4100
-Wire Wire Line
-	4650 4100 4650 4200
-$Comp
-L GND #PWR?
+$Comp
+L GND #PWR01
 U 1 1 57AA2B7C
 P 6800 3950
-F 0 "#PWR?" H 6800 3700 50  0001 C CNN
+F 0 "#PWR01" H 6800 3700 50  0001 C CNN
 F 1 "GND" H 6800 3800 50  0000 C CNN
 F 2 "" H 6800 3950 50  0000 C CNN
@@
 $EndComp
 $Comp
-L GND #PWR?
+L GND #PWR02
 U 1 1 57AA2B96
 P 4650 4500
-F 0 "#PWR?" H 4650 4250 50  0001 C CNN
+F 0 "#PWR02" H 4650 4250 50  0001 C CNN
 F 1 "GND" H 4650 4350 50  0000 C CNN
 F 2 "" H 4650 4500 50  0000 C CNN
@@
 $EndComp
 $Comp
-L +3.3V #PWR?
+L +3.3V #PWR03
 U 1 1 57AA2BB6
 P 6800 3750
-F 0 "#PWR?" H 6800 3600 50  0001 C CNN
+F 0 "#PWR03" H 6800 3600 50  0001 C CNN
 F 1 "+3.3V" H 6800 3890 50  0000 C CNN
 F 2 "" H 6800 3750 50  0000 C CNN
@@
 $EndComp
 $Comp
-L +3.3V #PWR?
+L +3.3V #PWR04
 U 1 1 57AA2BD0
 P 5650 3350
-F 0 "#PWR?" H 5650 3200 50  0001 C CNN
+F 0 "#PWR04" H 5650 3200 50  0001 C CNN
 F 1 "+3.3V" H 5650 3490 50  0000 C CNN
 F 2 "" H 5650 3350 50  0000 C CNN
@@
 NoConn ~ 4950 3500
 NoConn ~ 4950 3400
-Wire Wire Line
-	4650 4400 4650 4500
-Wire Wire Line
-	4650 4450 4950 4450
-Wire Wire Line
-	4950 4450 4950 4300
-Connection ~ 4650 4450
 Text GLabel 6350 3400 2    60   Input ~ 0
 OUT
@@
 CB
 $Comp
-L GND #PWR?
+L GND #PWR05
 U 1 1 57AA33D7
 P 5650 4350
-F 0 "#PWR?" H 5650 4100 50  0001 C CNN
+F 0 "#PWR05" H 5650 4100 50  0001 C CNN
 F 1 "GND" H 5650 4200 50  0000 C CNN
 F 2 "" H 5650 4350 50  0000 C CNN
@@
 	1    0    0    -1
 $EndComp
+$Comp
+L CONN_02X05 P1
+U 1 1 57AA3BC5
+P 3700 3550
+F 0 "P1" H 3700 3850 50  0000 C CNN
+F 1 "CONN_02X05" H 3700 3250 50  0000 C CNN
+F 2 "" H 3700 2350 50  0000 C CNN
+F 3 "" H 3700 2350 50  0000 C CNN
+	1    3700 3550
+	1    0    0    -1
+$EndComp
+Text GLabel 3700 3000 1    60   BiDi ~ 0
+OUT
+$Comp
+L +3.3V #PWR?
+U 1 1 57AA3C41
+P 4600 3750
+F 0 "#PWR?" H 4600 3600 50  0001 C CNN
+F 1 "+3.3V" H 4600 3890 50  0000 C CNN
+F 2 "" H 4600 3750 50  0000 C CNN
+F 3 "" H 4600 3750 50  0000 C CNN
+	1    4600 3750
+	1    0    0    -1
+$EndComp
+$Comp
+L GND #PWR?
+U 1 1 57AA3C5D
+P 2900 3750
+F 0 "#PWR?" H 2900 3500 50  0001 C CNN
+F 1 "GND" H 2900 3600 50  0000 C CNN
+F 2 "" H 2900 3750 50  0000 C CNN
+F 3 "" H 2900 3750 50  0000 C CNN
+	1    2900 3750
+	1    0    0    -1
+$EndComp
+$Comp
+L R_Small R1
+U 1 1 57AA3D48
+P 4050 3350
+F 0 "R1" V 4050 3300 50  0000 L CNN
+F 1 "100R" V 4050 3600 50  0000 L CNN
+F 2 "" H 4050 3350 50  0000 C CNN
+F 3 "" H 4050 3350 50  0000 C CNN
+	1    4050 3350
+	0    1    1    0
+$EndComp
+$Comp
+L R_Small R?
+U 1 1 57AA3E27
+P 4050 3450
+F 0 "R?" V 4050 3400 50  0000 L CNN
+F 1 "100R" V 4050 3700 50  0000 L CNN
+F 2 "" H 4050 3450 50  0000 C CNN
+F 3 "" H 4050 3450 50  0000 C CNN
+	1    4050 3450
+	0    1    1    0
+$EndComp
+$Comp
+L R_Small R?
+U 1 1 57AA3E6B
+P 4050 3550
+F 0 "R?" V 4050 3500 50  0000 L CNN
+F 1 "100R" V 4050 3800 50  0000 L CNN
+F 2 "" H 4050 3550 50  0000 C CNN
+F 3 "" H 4050 3550 50  0000 C CNN
+	1    4050 3550
+	0    1    1    0
+$EndComp
+$Comp
+L R_Small R?
+U 1 1 57AA3E9B
+P 4050 3650
+F 0 "R?" V 4050 3600 50  0000 L CNN
+F 1 "100R" V 4050 3900 50  0000 L CNN
+F 2 "" H 4050 3650 50  0000 C CNN
+F 3 "" H 4050 3650 50  0000 C CNN
+	1    4050 3650
+	0    1    1    0
+$EndComp
+$Comp
+L R_Small R?
+U 1 1 57AA3ED3
+P 3350 3350
+F 0 "R?" V 3350 3300 50  0000 L CNN
+F 1 "100R" V 3350 2900 50  0000 L CNN
+F 2 "" H 3350 3350 50  0000 C CNN
+F 3 "" H 3350 3350 50  0000 C CNN
+	1    3350 3350
+	0    1    1    0
+$EndComp
+$Comp
+L R_Small R?
+U 1 1 57AA3F18
+P 3350 3450
+F 0 "R?" V 3350 3400 50  0000 L CNN
+F 1 "100R" V 3350 3000 50  0000 L CNN
+F 2 "" H 3350 3450 50  0000 C CNN
+F 3 "" H 3350 3450 50  0000 C CNN
+	1    3350 3450
+	0    1    1    0
+$EndComp
+$Comp
+L R_Small R?
+U 1 1 57AA3F68
+P 3350 3550
+F 0 "R?" V 3350 3500 50  0000 L CNN
+F 1 "100R" V 3350 3100 50  0000 L CNN
+F 2 "" H 3350 3550 50  0000 C CNN
+F 3 "" H 3350 3550 50  0000 C CNN
+	1    3350 3550
+	0    1    1    0
+$EndComp
+$Comp
+L R_Small R?
+U 1 1 57AA3FAF
+P 3350 3650
+F 0 "R?" V 3350 3600 50  0000 L CNN
+F 1 "100R" V 3350 3200 50  0000 L CNN
+F 2 "" H 3350 3650 50  0000 C CNN
+F 3 "" H 3350 3650 50  0000 C CNN
+	1    3350 3650
+	0    1    1    0
+$EndComp
+Wire Wire Line
+	4950 4100 4650 4100
+Wire Wire Line
+	4650 4100 4650 4200
+Wire Wire Line
+	4650 4400 4650 4450
+Wire Wire Line
+	4650 4450 4650 4500
+Wire Wire Line
+	4650 4450 4950 4450
+Wire Wire Line
+	4950 4450 4950 4300
+Connection ~ 4650 4450
+Wire Wire Line
+	3450 3750 2900 3750
+Wire Wire Line
+	3950 3750 4600 3750
+Wire Wire Line
+	4200 3650 4150 3650
+Wire Wire Line
+	4200 3100 4200 3350
+Wire Wire Line
+	4200 3350 4200 3450
+Wire Wire Line
+	4200 3450 4200 3550
+Wire Wire Line
+	4200 3550 4200 3650
+Wire Wire Line
+	4200 3100 3700 3100
+Wire Wire Line
+	3700 3100 3200 3100
+Wire Wire Line
+	3200 3100 3200 3350
+Wire Wire Line
+	3200 3350 3200 3450
+Wire Wire Line
+	3200 3450 3200 3550
+Wire Wire Line
+	3200 3550 3200 3650
+Wire Wire Line
+	3200 3650 3250 3650
+Wire Wire Line
+	3250 3550 3200 3550
+Connection ~ 3200 3550
+Wire Wire Line
+	3250 3450 3200 3450
+Connection ~ 3200 3450
+Wire Wire Line
+	3250 3350 3200 3350
+Connection ~ 3200 3350
+Wire Wire Line
+	4150 3350 4200 3350
+Connection ~ 4200 3350
+Wire Wire Line
+	4150 3450 4200 3450
+Connection ~ 4200 3450
+Wire Wire Line
+	4150 3550 4200 3550
+Connection ~ 4200 3550
+Wire Wire Line
+	3700 3000 3700 3100
+Connection ~ 3700 3100
 $EndSCHEMATC

Commit message: annotated, footprints associated, netlist generated
Parts:
- C1: footprint (none) -> Capacitors_SMD:C_0805_HandSoldering
- IC1: footprint (none) -> SMD_Packages:SO-16-N
- P1: footprint (none) -> Connect:IDC_Header_Straight_10pins
- R1: footprint (none) -> Resistors_SMD:R_0805_HandSoldering
- R2, R3, R4, R5, R6, R7, R8: renamed from R?; footprint (none) -> Resistors_SMD:R_0805_HandSoldering
- Rvco1: renamed from R1; footprint (none) -> Diodes_SMD:MiniMELF_Handsoldering
Changed lines of the file:
@@
 F 0 "C1" H 6810 3920 50  0000 L CNN
 F 1 "100n" H 6810 3770 50  0000 L CNN
-F 2 "" H 6800 3850 50  0000 C CNN
+F 2 "Capacitors_SMD:C_0805_HandSoldering" H 6800 3850 50  0001 C CNN
 F 3 "" H 6800 3850 50  0000 C CNN
 	1    6800 3850
@@
 $EndComp
 $Comp
-L R_Small R1
+L R_Small Rvco1
 U 1 1 57AA2285
 P 4650 4300
-F 0 "R1" H 4680 4320 50  0000 L CNN
+F 0 "Rvco1" H 4680 4320 50  0000 L CNN
 F 1 "220K" H 4680 4260 50  0000 L CNN
-F 2 "" H 4650 4300 50  0000 C CNN
+F 2 "Diodes_SMD:MiniMELF_Handsoldering" H 4650 4300 50  0001 C CNN
 F 3 "" H 4650 4300 50  0000 C CNN
 	1    4650 4300
@@
 F 0 "IC1" H 5650 3700 50  0000 C CNN
 F 1 "4046" H 5650 3900 50  0000 C CNN
-F 2 "" H 5650 3800 60  0000 C CNN
+F 2 "SMD_Packages:SO-16-N" H 5650 3800 60  0001 C CNN
 F 3 "" H 5650 3800 60  0000 C CNN
 	1    5650 3800
@@
 F 0 "P1" H 3700 3850 50  0000 C CNN
 F 1 "CONN_02X05" H 3700 3250 50  0000 C CNN
-F 2 "" H 3700 2350 50  0000 C CNN
+F 2 "Connect:IDC_Header_Straight_10pins" H 3700 2350 50  0001 C CNN
 F 3 "" H 3700 2350 50  0000 C CNN
 	1    3700 3550
@@
 OUT
 $Comp
-L +3.3V #PWR?
+L +3.3V #PWR06
 U 1 1 57AA3C41
 P 4600 3750
-F 0 "#PWR?" H 4600 3600 50  0001 C CNN
+F 0 "#PWR06" H 4600 3600 50  0001 C CNN
 F 1 "+3.3V" H 4600 3890 50  0000 C CNN
 F 2 "" H 4600 3750 50  0000 C CNN
@@
 $EndComp
 $Comp
-L GND #PWR?
+L GND #PWR07
 U 1 1 57AA3C5D
 P 2900 3750
-F 0 "#PWR?" H 2900 3500 50  0001 C CNN
+F 0 "#PWR07" H 2900 3500 50  0001 C CNN
 F 1 "GND" H 2900 3600 50  0000 C CNN
 F 2 "" H 2900 3750 50  0000 C CNN
@@
 F 0 "R1" V 4050 3300 50  0000 L CNN
 F 1 "100R" V 4050 3600 50  0000 L CNN
-F 2 "" H 4050 3350 50  0000 C CNN
+F 2 "Resistors_SMD:R_0805_HandSoldering" H 4050 3350 50  0001 C CNN
 F 3 "" H 4050 3350 50  0000 C CNN
 	1    4050 3350
@@
 $EndComp
 $Comp
-L R_Small R?
+L R_Small R6
 U 1 1 57AA3E27
 P 4050 3450
-F 0 "R?" V 4050 3400 50  0000 L CNN
+F 0 "R6" V 4050 3400 50  0000 L CNN
 F 1 "100R" V 4050 3700 50  0000 L CNN
-F 2 "" H 4050 3450 50  0000 C CNN
+F 2 "Resistors_SMD:R_0805_HandSoldering" H 4050 3450 50  0001 C CNN
 F 3 "" H 4050 3450 50  0000 C CNN
 	1    4050 3450
@@
 $EndComp
 $Comp
-L R_Small R?
+L R_Small R7
 U 1 1 57AA3E6B
 P 4050 3550
-F 0 "R?" V 4050 3500 50  0000 L CNN
+F 0 "R7" V 4050 3500 50  0000 L CNN
 F 1 "100R" V 4050 3800 50  0000 L CNN
-F 2 "" H 4050 3550 50  0000 C CNN
+F 2 "Resistors_SMD:R_0805_HandSoldering" H 4050 3550 50  0001 C CNN
 F 3 "" H 4050 3550 50  0000 C CNN
 	1    4050 3550
@@
 $EndComp
 $Comp
-L R_Small R?
+L R_Small R8
 U 1 1 57AA3E9B
 P 4050 3650
-F 0 "R?" V 4050 3600 50  0000 L CNN
+F 0 "R8" V 4050 3600 50  0000 L CNN
 F 1 "100R" V 4050 3900 50  0000 L CNN
-F 2 "" H 4050 3650 50  0000 C CNN
+F 2 "Resistors_SMD:R_0805_HandSoldering" H 4050 3650 50  0001 C CNN
 F 3 "" H 4050 3650 50  0000 C CNN
 	1    4050 3650
@@
 $EndComp
 $Comp
-L R_Small R?
+L R_Small R2
 U 1 1 57AA3ED3
 P 3350 3350
-F 0 "R?" V 3350 3300 50  0000 L CNN
+F 0 "R2" V 3350 3300 50  0000 L CNN
 F 1 "100R" V 3350 2900 50  0000 L CNN
-F 2 "" H 3350 3350 50  0000 C CNN
+F 2 "Resistors_SMD:R_0805_HandSoldering" H 3350 3350 50  0001 C CNN
 F 3 "" H 3350 3350 50  0000 C CNN
 	1    3350 3350
@@
 $EndComp
 $Comp
-L R_Small R?
+L R_Small R3
 U 1 1 57AA3F18
 P 3350 3450
-F 0 "R?" V 3350 3400 50  0000 L CNN
+F 0 "R3" V 3350 3400 50  0000 L CNN
 F 1 "100R" V 3350 3000 50  0000 L CNN
-F 2 "" H 3350 3450 50  0000 C CNN
+F 2 "Resistors_SMD:R_0805_HandSoldering" H 3350 3450 50  0001 C CNN
 F 3 "" H 3350 3450 50  0000 C CNN
 	1    3350 3450
@@
 $EndComp
 $Comp
-L R_Small R?
+L R_Small R4
 U 1 1 57AA3F68
 P 3350 3550
-F 0 "R?" V 3350 3500 50  0000 L CNN
+F 0 "R4" V 3350 3500 50  0000 L CNN
 F 1 "100R" V 3350 3100 50  0000 L CNN
-F 2 "" H 3350 3550 50  0000 C CNN
+F 2 "Resistors_SMD:R_0805_HandSoldering" H 3350 3550 50  0001 C CNN
 F 3 "" H 3350 3550 50  0000 C CNN
 	1    3350 3550
@@
 $EndComp
 $Comp
-L R_Small R?
+L R_Small R5
 U 1 1 57AA3FAF
 P 3350 3650
-F 0 "R?" V 3350 3600 50  0000 L CNN
+F 0 "R5" V 3350 3600 50  0000 L CNN
 F 1 "100R" V 3350 3200 50  0000 L CNN
-F 2 "" H 3350 3650 50  0000 C CNN
+F 2 "Resistors_SMD:R_0805_HandSoldering" H 3350 3650 50  0001 C CNN
 F 3 "" H 3350 3650 50  0000 C CNN
 	1    3350 3650
@@
 	4650 4100 4650 4200
 Wire Wire Line
-	4650 4400 4650 4450
-Wire Wire Line
-	4650 4450 4650 4500
+	4650 4400 4650 4500
 Wire Wire Line
 	4650 4450 4950 4450
@@
 	4200 3650 4150 3650
 Wire Wire Line
-	4200 3100 4200 3350
-Wire Wire Line
-	4200 3350 4200 3450
-Wire Wire Line
-	4200 3450 4200 3550
-Wire Wire Line
-	4200 3550 4200 3650
-Wire Wire Line
-	4200 3100 3700 3100
-Wire Wire Line
-	3700 3100 3200 3100
-Wire Wire Line
-	3200 3100 3200 3350
-Wire Wire Line
-	3200 3350 3200 3450
-Wire Wire Line
-	3200 3450 3200 3550
-Wire Wire Line
-	3200 3550 3200 3650
+	4200 3100 4200 3650
+Wire Wire Line
+	3200 3100 4200 3100
+Wire Wire Line
+	3200 3100 3200 3650
 Wire Wire Line
 	3200 3650 3250 3650
